Commit message: modified servo

File: sawyer_moveit_config/srdf/sawyer_base.srdf.xacro (robot description, xacro)
@@ -33,4 +33,22 @@
         <joint name="right_j4" value="0" />
         <joint name="right_j5" value="0" />
+        <joint name="right_j6" value="0" />
+    </group_state>
+    <group_state name="folded" group="right_arm">
+        <joint name="right_j0" value="0" />
+        <joint name="right_j1" value="-1.57" />
+        <joint name="right_j2" value="0" />
+        <joint name="right_j3" value="-1.57" />
+        <joint name="right_j4" value="0" />
+        <joint name="right_j5" value="1.57" />
+        <joint name="right_j6" value="0" />
+    </group_state>
+    <group_state name="home" group="right_arm">
+        <joint name="right_j0" value="0" />
+        <joint name="right_j1" value="-0.9" />
+        <joint name="right_j2" value="0" />
+        <joint name="right_j3" value="1.8" />
+        <joint name="right_j4" value="0" />
+        <joint name="right_j5" value="-0.9" />
         <joint name="right_j6" value="0" />
     </group_state>
